Commit message: update tm{12,5}_description packages to accept a kinematics file
I.e., the type of kinematics file created by tm_calibration. This
involves editing the tmX_upload.launch and related
tmX{_robot}.urdf.xacro files.

Since the visual/collision meshes are not oriented in the same way as
the kinematics tree, this required adding visual/collision origins for
the majority of links.

Once the description packages are merged to one, duplication can be
reduced by a lot.

File: tm5_description/urdf/tm5_900.urdf.xacro (robot description, xacro)
@@ -31,5 +31,6 @@
     transmission_hw_interface:=hardware_interface/PositionJointInterface
     safety_limits:=false safety_pos_margin:=0.15
-    safety_k_position:=20">
+    safety_k_position:=20 kinematics_file">
+    <xacro:property name="kinematics" value="${kinematics_file['kinematics']}"/>
     <!-- Inertia parameters -->
     <xacro:property name="base_mass" value="1.0" />
@@ -79,4 +80,5 @@
     <link name="${prefix}base_link" >
       <visual>
+        <origin xyz="0 0 0" rpy="${pi / 2.0} 0 0"/>
         <geometry>
         <xacro:unless value="${stl_mesh}">
@@ -92,4 +94,5 @@
       </visual>
       <collision>
+        <origin xyz="0 0 0" rpy="${pi / 2.0} 0 0"/>
         <geometry>
           <mesh filename="package://tm5_description/meshes/tm5_900/collision/tm5_base_c.STL" />
@@ -103,6 +106,6 @@
       <parent link="${prefix}base_link" />
       <child link = "${prefix}shoulder_1_link" />
-      <origin xyz="0 ${shoulder_height} 0" rpy="0 0 0" />
-      <axis xyz="0 1 0" />
+      <origin xyz="${kinematics['shoulder_1']['x']} ${kinematics['shoulder_1']['y']} ${kinematics['shoulder_1']['z']}" rpy="${kinematics['shoulder_1']['roll']} ${kinematics['shoulder_1']['pitch']} ${kinematics['shoulder_1']['yaw']}" />
+      <axis xyz="0 0 1" />
       <limit lower="${shoulder_1_lower_limit}" upper="${shoulder_1_upper_limit}" effort="150.0" velocity="3.15" />
       <xacro:if value="${safety_limits}">
@@ -113,4 +116,5 @@
     <link name="${prefix}shoulder_1_link">
       <visual>
+        <origin xyz="0 0 0" rpy="${pi / 2.0} 0 0"/>
         <geometry>
         <xacro:unless value="${stl_mesh}">
@@ -126,4 +130,5 @@
       </visual>
       <collision>
+        <origin xyz="0 0 0" rpy="${pi / 2.0} 0 0"/>
         <geometry>
           <mesh filename="package://tm5_description/meshes/tm5_900/collision/tm_400w_01_c.STL" />
@@ -137,6 +142,6 @@
       <parent link="${prefix}shoulder_1_link" />
       <child link = "${prefix}arm_1_link" />
-      <origin xyz="0 0 ${shoulder_offset}" rpy="0 0 0" />
-      <axis xyz="0 0 -1" />
+      <origin xyz="${kinematics['shoulder_2']['x']} ${kinematics['shoulder_2']['y']} ${kinematics['shoulder_2']['z']}" rpy="${kinematics['shoulder_2']['roll']} ${kinematics['shoulder_2']['pitch']} ${kinematics['shoulder_2']['yaw']}" />
+      <axis xyz="0 0 1" />
       <limit lower="${shoulder_2_lower_limit}" upper="${shoulder_2_upper_limit}" effort="150.0" velocity="3.15" />
       <xacro:if value="${safety_limits}">
@@ -147,4 +152,5 @@
     <link name="${prefix}arm_1_link">
       <visual>
+        <origin xyz="0 0 -${shoulder_offset}" rpy="0 3.141592653589793 -${pi / 2.0}"/>
         <geometry>
         <xacro:unless value="${stl_mesh}">
@@ -160,4 +166,5 @@
       </visual>
       <collision>
+        <origin xyz="0 0 -${shoulder_offset}" rpy="0 3.141592653589793 -${pi / 2.0}"/>
         <geometry>
           <mesh filename="package://tm5_description/meshes/tm5_900/collision/tm5_900_arm1_c.STL" />
@@ -171,6 +178,6 @@
       <parent link="${prefix}arm_1_link" />
       <child link = "${prefix}arm_2_link" />
-      <origin xyz="0 ${arm_1_length} ${-elbow_offset}" rpy="0 0 0" />
-      <axis xyz="0 0 -1" />
+      <origin xyz="${kinematics['elbow']['x']} ${kinematics['elbow']['y']} ${kinematics['elbow']['z']}" rpy="${kinematics['elbow']['roll']} ${kinematics['elbow']['pitch']} ${kinematics['elbow']['yaw']}" />
+      <axis xyz="0 0 1" />
       <limit lower="${elbow_lower_limit}" upper="${elbow_upper_limit}" effort="150.0" velocity="3.15" />
       <xacro:if value="${safety_limits}">
@@ -181,4 +188,5 @@
     <link name="${prefix}arm_2_link">
       <visual>
+        <origin xyz="0 0 -${shoulder_offset - elbow_offset}" rpy="0 3.141592653589793 -${pi / 2.0}"/>
         <geometry>
         <xacro:unless value="${stl_mesh}">
@@ -194,4 +202,5 @@
       </visual>
       <collision>
+        <origin xyz="0 0 -${shoulder_offset - elbow_offset}" rpy="0 3.141592653589793 -${pi / 2.0}"/>
         <geometry>
           <mesh filename="package://tm5_description/meshes/tm5_900/collision/tm5_900_arm2_c.STL" />
@@ -205,6 +214,6 @@
       <parent link="${prefix}arm_2_link" />
       <child link = "${prefix}wrist_1_link" />
-      <origin xyz="0 ${arm_2_length} ${wrist_offset}" rpy="0 0 0" />
-      <axis xyz="0 0 -1" />
+      <origin xyz="${kinematics['wrist_1']['x']} ${kinematics['wrist_1']['y']} ${kinematics['wrist_1']['z']}" rpy="${kinematics['wrist_1']['roll']} ${kinematics['wrist_1']['pitch']} ${kinematics['wrist_1']['yaw']}" />
+      <axis xyz="0 0 1" />
       <limit lower="${wrist_1_lower_limit}" upper="${wrist_1_upper_limit}" effort="150.0" velocity="3.15"/>
       <xacro:if value="${safety_limits}">
@@ -215,4 +224,5 @@
     <link name="${prefix}wrist_1_link">
       <visual>
+        <origin xyz="0 0 0" rpy="${pi} 0 0"/>
         <geometry>
         <xacro:unless value="${stl_mesh}">
@@ -228,4 +238,5 @@
       </visual>
       <collision>
+        <origin xyz="0 0 0" rpy="${pi} 0 0"/>
         <geometry>
           <mesh filename="package://tm5_description/meshes/tm5_900/collision/tm_100w_01_c.STL" />
@@ -239,6 +250,6 @@
       <parent link="${prefix}wrist_1_link" />
       <child link = "${prefix}wrist_2_link" />
-      <origin xyz="0 ${wrist_2_length} 0" rpy="0 0 0" />
-      <axis xyz="0 1 0" />
+      <origin xyz="${kinematics['wrist_2']['x']} ${kinematics['wrist_2']['y']} ${kinematics['wrist_2']['z']}" rpy="${kinematics['wrist_2']['roll']} ${kinematics['wrist_2']['pitch']} ${kinematics['wrist_2']['yaw']}" />
+      <axis xyz="0 0 1" />
       <limit lower="${wrist_2_lower_limit}" upper="${wrist_2_upper_limit}" effort="150.0" velocity="3.15" />
       <xacro:if value="${safety_limits}">
@@ -249,4 +260,5 @@
     <link name="${prefix}wrist_2_link">
       <visual>
+        <origin xyz="0 0 0" rpy="${pi / 2.0} 0 0"/>
         <geometry>
         <xacro:unless value="${stl_mesh}">
@@ -262,4 +274,5 @@
       </visual>
       <collision>
+        <origin xyz="0 0 0" rpy="${pi / 2.0} 0 0"/>
         <geometry>
           <mesh filename="package://tm5_description/meshes/tm5_900/collision/tm_100w_02_c.stl" />
@@ -273,5 +286,5 @@
       <parent link="${prefix}wrist_2_link" />
       <child link = "${prefix}wrist_3_link" />
-      <origin xyz="0 0 ${wrist_3_length}" rpy="0 0 0" />
+      <origin xyz="${kinematics['wrist_3']['x']} ${kinematics['wrist_3']['y']} ${kinematics['wrist_3']['z']}" rpy="${kinematics['wrist_3']['roll']} ${kinematics['wrist_3']['pitch']} ${kinematics['wrist_3']['yaw']}" />
       <axis xyz="0 0 1" />
       <limit lower="${wrist_3_lower_limit}" upper="${wrist_3_upper_limit}" effort="150.0" velocity="3.15" />
@@ -316,5 +329,5 @@
       <parent link="${prefix}base" />
       <child link="${prefix}base_link" />
-      <origin xyz="0 0 0" rpy="${0.5 * pi} 0 0" /> <!-- Note: 0.5 * pi -->
+      <origin xyz="0 0 0" rpy="0 0 0" />
     </joint>
     <!-- Frame coincident with all-zeros TCP on TM controller -->

File: tm5_description/urdf/tm5_900_robot.urdf.xacro (robot description, xacro)
@@ -9,5 +9,6 @@
   <!-- arm -->
   <!--xacro:tm5_900_robot prefix="" joint_limited="false" transmission_hw_interface="$(arg transmission_hw_interface)" /-->
-  <xacro:tm5_900_robot prefix="" joint_limited="false" stl_mesh="$(arg stl_mesh)" />
+  <xacro:arg name="kinematics_config" default="$(find tm5_description)/config/tm5_900_default.yaml" />
+  <xacro:tm5_900_robot prefix="" joint_limited="false" stl_mesh="$(arg stl_mesh)" kinematics_file="${load_yaml('$(arg kinematics_config)')}" />
   <link name="world" />
   <joint name="world_joint" type="fixed">
